File: MSP430AFE253_Demo_Board.sch (KiCad schematic (older format))
At the start: 45 parts, among them J1 USB_MINI_B, P1 POWER, P2 3.3V, P3 HEADER_1X4, P4 TX, P5 RX, P6 DEBUG, SW1 FSM4JH, SW2 FSM4JH, SW3 FSM4JH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

Commit message: Updated per VCC track change to route track through middle of RX & TX header pins instead of around outside near PCB edge.
Connections:
- wire segments 181 -> 179
- no-connect marks 0 -> 1
Changed lines of the file:
@@
-EESchema Schematic File Version 2  date 9/13/2012 3:38:11 PM
+EESchema Schematic File Version 2  date 9/28/2012 7:27:18 PM
 LIBS:power
 LIBS:device
@@
 Sheet 1 1
 Title ""
-Date "13 sep 2012"
+Date "29 sep 2012"
 Rev ""
 Comp ""
@@
 Comment4 ""
 $EndDescr
+NoConn ~ 3550 900
 Text Notes 7525 3725 0    40   ~ 0
 GND
@@
 Wire Wire Line
 	950  1300 1050 1300
-Wire Wire Line
-	3550 900  3550 950
 Connection ~ 2700 1050
 Wire Wire Line
@@
 	3400 1050 3400 900
 Wire Wire Line
-	3550 950  3600 950
-Connection ~ 3600 950
-Wire Wire Line
 	4600 2750 4600 2850
