File: Hardware/KiCAD_Project_Files/MSP430AFE253_Demo_Board.sch (KiCad schematic (older format))
At the start: 45 parts, among them J1 USB_MINI_B, P1 POWER, P2 3.3V, P3 HEADER_1X4, P4 TX, P5 RX, P6 DEBUG, SW1 FSM4JH, SW2 FSM4JH, SW3 FSM4JH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

Commit message: Rev'd board design and schematic to utilize smaller-footprint 8MHz crystal resonators.
Parts:
- X1: value 4MHz -> 8MHz
- X2: value 3.686MHz -> 8MHz
Changed lines of the file:
@@
-EESchema Schematic File Version 2  date 9/28/2012 7:27:18 PM
+EESchema Schematic File Version 2  date 12/5/2012 8:16:33 PM
 LIBS:power
 LIBS:device
@@
 Sheet 1 1
 Title ""
-Date "29 sep 2012"
+Date "6 dec 2012"
 Rev ""
 Comp ""
@@
 P 3500 3600
 F 0 "X1" H 3500 3700 40  0000 C CNN
-F 1 "4MHz" H 3600 3500 40  0000 C CNN
+F 1 "8MHz" H 3600 3500 40  0000 C CNN
 	1    3500 3600
 	1    0    0    -1
@@
 P 8150 4850
 F 0 "X2" H 8150 4950 40  0000 C CNN
-F 1 "3.686MHz" H 8350 4750 40  0000 C CNN
+F 1 "8MHz" H 8350 4750 40  0000 C CNN
 	1    8150 4850
 	1    0    0    -1
