File: Hardware/KiCAD_Project_Files/MSP430AFE253_Demo_Board.sch (KiCad schematic (older format))
At the start: 45 parts, among them J1 USB_MINI_B, P1 POWER, P2 3.3V, P3 HEADER_1X4, P4 TX, P5 RX, P6 DEBUG, SW1 FSM4JH, SW2 FSM4JH, SW3 FSM4JH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

Commit message: The Freescale USB-to-Serial IC seems to be obsolee.  This is a baseline check-in before changing to the FTDI FT230XQ.
Other:
- note removed: "MSP430AFE253 Demo Board"
- moved on the sheet: C1, C10, C2, C3, C4, C5, C6, C7, C8, C9, D1, D2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

Commit message: Rev 3 release
Parts:
- removed C4, C7, C8: 4.7u, symbol CAPP
- removed R4, R5: 47k, symbol RES_SMALL
- removed R6, R8: 0, symbol RES_SMALL
- removed R7: 1M, symbol RES_SMALL
- removed SW1, SW2, SW3: FSM4JH, symbol FSM4JH
- removed U1: USB2SERA10CFK, symbol USB2SERA10CFK
- removed X1: 8MHz, symbol CERAMIC_RESONATOR
- added C11, C13: 0.1u, symbol CAP
- added C12, C4, C7, C8: 4.7u, symbol CAP
- added SW1, SW2, SW3: FSMSM, symbol FSMSM
- added U1: FT230XQ, symbol FT230XQ
- C1, C10, C2, C5, C6, C9: value .1u -> 0.1u
- C3: value .1u -> 4.7u
- X2: value 8MHz -> 3.68MHz
Connections:
- net labels removed: EXTAL, XTAL
- wire segments 179 -> 169
- no-connect marks 1 -> 5
Other:
- moved on the sheet: C5, C6, D1, D2
