File: Hardware/KiCAD_Project_Files/MSP430AFE253_Demo_Board.sch (KiCad schematic (older format))
At the start: 42 parts, among them J1 USB_MINI_B, P1 POWER, P2 3.3V, P3 HEADER_1X4, P4 TX, P5 RX, P6 DEBUG, SW1 FSMSM, SW2 FSMSM, SW3 FSMSM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

Commit message: First commit at Rev 4
Other:
- note added: "RX"
- note added: "TX"
Changed lines of the file:
@@
 Title "MSP430AFE253 Demo Board"
 Date "Saturday, July 26, 2014"
-Rev "3"
+Rev "4"
 Comp "Casco Logix"
 Comment1 ""
@@
 P 6500 3600
 F 0 "#PWR01" H 6500 3700 30  0001 C CNN
-F 1 "VCC" H 6500 3700 30  0000 C CNN
+F 1 "VCC" H 6500 3700 40  0000 C CNN
 F 2 "" H 6500 3600 60  0001 C CNN
 F 3 "" H 6500 3600 60  0001 C CNN
@@
 P 6200 3600
 F 0 "#PWR06" H 6200 3700 30  0001 C CNN
-F 1 "VCC" H 6200 3700 30  0000 C CNN
+F 1 "VCC" H 6200 3700 40  0000 C CNN
 F 2 "" H 6200 3600 60  0001 C CNN
 F 3 "" H 6200 3600 60  0001 C CNN
@@
 P 1150 1100
 F 0 "#PWR019" H 1150 1190 20  0001 C CNN
-F 1 "VBUS" H 1150 1190 30  0000 C CNN
+F 1 "VBUS" H 1150 1200 40  0000 C CNN
 F 2 "" H 1150 1100 60  0001 C CNN
 F 3 "" H 1150 1100 60  0001 C CNN
@@
 P 1200 4000
 F 0 "#PWR022" H 1200 4100 30  0001 C CNN
-F 1 "VCC" H 1200 4100 30  0000 C CNN
+F 1 "VCC" H 1200 4100 40  0000 C CNN
 F 2 "" H 1200 4000 60  0001 C CNN
 F 3 "" H 1200 4000 60  0001 C CNN
@@
 P 8450 4950
 F 0 "#PWR023" H 8450 5050 30  0001 C CNN
-F 1 "VCC" H 8450 5050 30  0000 C CNN
+F 1 "VCC" H 8450 5050 40  0000 C CNN
 F 2 "" H 8450 4950 60  0001 C CNN
 F 3 "" H 8450 4950 60  0001 C CNN
@@
 P 5750 1000
 F 0 "#PWR024" H 5750 1100 30  0001 C CNN
-F 1 "VCC" H 5750 1100 30  0000 C CNN
+F 1 "VCC" H 5750 1100 40  0000 C CNN
 F 2 "" H 5750 1000 60  0001 C CNN
 F 3 "" H 5750 1000 60  0001 C CNN
@@
 P 3600 700
 F 0 "#PWR025" H 3600 800 30  0001 C CNN
-F 1 "VCC" H 3600 800 30  0000 C CNN
+F 1 "VCC" H 3600 800 40  0000 C CNN
 F 2 "" H 3600 700 60  0001 C CNN
 F 3 "" H 3600 700 60  0001 C CNN
@@
 NoConn ~ 3450 2000
 NoConn ~ 3450 2700
-NoConn ~ 3450 2600
 $Comp
 L CAP C1
@@
 Wire Wire Line
 	3450 2500 4100 2500
-Wire Wire Line
-	3700 2400 3700 2950
-Wire Wire Line
-	3450 2400 3700 2400
 Connection ~ 2850 2950
 Wire Wire Line
@@
 	1    0    0    -1
 $EndComp
+Text Notes 4200 3150 0    40   ~ 0
+RX
+Text Notes 3800 3150 0    40   ~ 0
+TX
+Wire Wire Line
+	3450 2600 3700 2600
+Wire Wire Line
+	3700 2600 3700 2950
+NoConn ~ 3450 2400
 $EndSCHEMATC

Commit message: Check in current state of Rev 4 design (in-progress) before checking out and forking the Rev 1 design.
Parts:
- added R4, R5, R6, R7: 1k, symbol RES_SMALL
- R1, R2: value 1.8k -> 270
- R15, R16: value 47k -> 1
- X2: value 3.68MHz -> 8MHz
Connections:
- wire segments 169 -> 173
Other:
- note removed: "RX"
- note removed: "TX"
- moved on the sheet: C10, C9

Commit message: Final commit for Rev4 release
Parts:
- removed C10, C9: 0.1u, symbol CAP
- removed R15, R16: 1, symbol RES_SMALL
- removed R4, R5, R6, R7: 1k, symbol RES_SMALL
- added TP1, TP2, TP3, TP4: 5015, symbol 5015
Connections:
- wire segments 173 -> 163
- no-connect marks 5 -> 1
Other:
- moved on the sheet: D1, D2, D3, SW1, SW2

Commit message: Rev 5 Commit. Generated new board gerbers and drawings. Updated user guide documentation and board renderings.
Parts:
- D1: value GREEN -> GRN
Connections:
- net labels added: VCCIO
- wire segments 163 -> 191
